File: hardware/daughtercard/daughtercard.kicad_pcb (KiCad board)
At the start: 2 copper layers, 74 x 60 mm, 52 parts, among them J1 Anzeige, J2 Bus in, J3 Bus out, J4 42V~ in, J5 42V~ out, J6 UPDI, Q1 BSS84, Q2 MMBT3904, Q3 MMBT3904, U1 ATtiny1616-SNR, U2 TP8485E-SR

Commit message: JLCPCB-Bestueckung vorbereitet: LCSC-Nummern, --jlc-Export, R16 0805
- LCSC-Dict in gen_daughtercard_sch.py: Basic Parts, wo moeglich (alle
  0805/1206-R und -C, MMBT3904). Nur U1, U2 und BAT54S bleiben Extended.
- gen_daughtercard_pcb.py --jlc: erzeugt jlc/BOM.csv + jlc/CPL.csv im
  JLCPCB-Format (gitignored, Bauartefakt). Schliesst #, H*, TP*, JP*,
  J1-J6 (Handloetung) und DNP (Q3, R10) aus.
- R16 von 1206 auf 0805 (D-1): 120 Ohm gibt es bei JLCPCB nur in 0805
  als Basic Part; Verlustleistung ~50 mW unkritisch. Schaltplan und PCB
  neu erzeugt, ERC 0/0, DRC unveraendert (4 enge Nachbarpaare am
  Bus-Stecker, vom Nutzer zu justieren).
- docs/jlc-bestueckung.md: Stueckliste mit LCSC-Zuordnung, zweite
  Anschlussbild-Pruefung aller Symbole (ohne Befund: MMBT3904, BSS84,
  BAT54S, TP8485E, ATtiny1616), Ruestkosten-Bilanz, offene
  Entscheidungen D-2 (C3), D-3 (F1), D-4 (Q1-LCSC).
- schaltplan-daughtercard.md v0.4, projektstand.md, toolchain.md.

Co-Authored-By: Claude Sonnet 5 <noreply@anthropic.com>
Claude-Session: https://claude.ai/code/session_01UsXTvE3jGgoK5Hec7hVbyD
Parts:
- R16: footprint R_1206_3216Metric -> R_0805_2012Metric

Commit message: J1 von Wannenstecker auf Buchsenleiste 2x5 (board-to-board)
Die Daughter Card wird huckepack direkt auf den Pfostenstecker der
Anzeigenplatine gesteckt (Ruecksprache 31.08.2026). Ein Wannenstecker
(Stifte im Kragen) passt dort nicht - richtig ist eine Buchsenleiste.

- Footprint J1: Connector_IDC:IDC-Header_2x05_P2.54mm_Vertical
  -> Connector_PinSocket_2.54mm:PinSocket_2x05_P2.54mm_Vertical
  (Referenz BKL 10120960). Pinbelegung 1..10 unveraendert.
- J1 ist damit NICHT mehr mechanisch kodiert. Pin 2/4 fuehren 42 V~;
  180-Grad-verdreht aufgesteckt zerstoert das U1/U2/Q1/Q2. Abgesichert
  ueber Mechanik (offen: J1-M), Bestueckungsdruck und Durchgangspruefung.
- docs/pruefpunkte-j1-buchsenleiste.md: Bewertung, Absicherung, Freigabe,
  offener Punkt J1-M (mechanische Kodierung der Drehlage).
- Schaltplan v0.5 (4.1 Verpol-Hinweis, 3.3, Pruefliste 9.1),
  Spezifikation v0.8 (4.6), layout-daughtercard.md (Checkliste, AC-Zone,
  Courtyard-Notiz), projektstand.md.
- Schaltplan + PCB neu erzeugt, ERC 0/0, DRC unveraendert (4 enge Paare
  am Bus-Stecker J2/J3, nichts an J1).

Co-Authored-By: Claude Sonnet 5 <noreply@anthropic.com>
Claude-Session: https://claude.ai/code/session_01UsXTvE3jGgoK5Hec7hVbyD
Parts:
- J1: footprint IDC-Header_2x05_P2.54mm_Vertical -> PinSocket_2x05_P2.54mm_Vertical
