File: hardware/daughtercard/daughtercard.kicad_pcb (KiCad board)
At the start: 2 copper layers, 74 x 60 mm, 52 parts, among them J1 Anzeige, J2 Bus in, J3 Bus out, J4 42V~ in, J5 42V~ out, J6 UPDI, Q1 BSS84, Q2 MMBT3904, Q3 MMBT3904, U1 ATtiny1616-SNR, U2 TP8485E-SR

Commit message: PCB gerouted: alle Bahnen 0,5 mm ausser AC, schwarze Platine, Maker-Mark
Routing-Lauf auf der Betreiber-Platzierung (J1-J5 fix). FreeRouting 2.3.0
plus tools/finish_routes.py fuer die 1-2 Verbindungen, die FreeRouting
offen laesst (Rastersuch-Router). Masseflaeche F.Cu + B.Cu mit
Stitching-Raster und je einem Via an jedem GND-Pad.

Netzklassen (Betreiber-Vorgabe):
- alle Leiterbahnen 0,5 mm (an SOIC-Pins auf 0,375 mm verjuengt)
- nur AC1/AC2 1,5 mm
- GND ueber die Flaeche
Konsequenz +5V-Spannungsabfall bei 10 Modulen -> docs/jlc-bestueckung.md D-5.

Platzierung angepasst (ausserhalb J1-J5, vom Betreiber freigegeben):
- F1 von PTC 0,5 A auf 0-Ohm-Bruecke (R_1206 / 0R / C17888, D-3):
  F1 liegt im +5V-Durchgangspfad, ein PTC wuerde bei 10 Modulen ausloesen
- Q1-Q3, R7-R10, Status-LED aus dem AC-Korridor nach rechts gerueckt
  -> AC-Bahn haelt danach >= 0,55 mm Kupfer zu jeder Logikbahn
- J6 (UPDI) unter U1

Schaltplan: F1 -> krone:R "0R"; Footprint-Pfade der .kicad_pcb per
UUID-Remapping auf den neu erzeugten Schaltplan gezogen (Platzierung und
Routing bleiben erhalten). ERC 0/0, DRC 0/0.

Fertigung:
- Lagenaufbau schwarze Loetstoppmaske / weisser Bestueckungsdruck
- Maker-Kennzeichnung auf B.SilkS: GitHub-Marke (octicon mark-github, aus
  SVG getraced, footprints/logos.pretty/Logo_GitHub) + Text "TenOfNine"
- tools/add_silk_marks.py setzt beides idempotent

Neu: tools/finish_routes.py, tools/add_silk_marks.py, fp-lib-table,
footprints/logos.pretty/. setup.sh: python3-numpy fuer finish_routes.
Schaltplan v0.7, Doku (Layout, JLC, Toolchain, Projektstand) fortgeschrieben.

Co-Authored-By: Claude Sonnet 5 <noreply@anthropic.com>
Claude-Session: https://claude.ai/code/session_01UsXTvE3jGgoK5Hec7hVbyD
Parts:
- added GH1: Logo_GitHub, Logo_GitHub, B.Cu at (34.0, 25.0)
- F1: value 500mA -> 0R; footprint Fuse_1206_3216Metric -> R_1206_3216Metric
- moved J6 28.4 mm to (39.0, 51.0), turned to 0 degrees
- moved R8 15.5 mm to (65.0, 16.0)
- moved R15 14.0 mm to (61.0, 29.5)
- moved D4 14.0 mm to (65.5, 29.5)
- moved Q2 12.2 mm to (62.0, 25.0)
- moved Q1 11.1 mm to (66.0, 25.0)
- moved Q3 10.1 mm to (70.0, 25.0)
- moved R9 9.85 mm to (69.0, 16.0)
- moved R7 7.21 mm to (61.0, 16.0)
- moved R10 4.00 mm to (61.0, 20.0)
Routing:
- net /+5V: track 0.00 -> 142.6 mm, vias 0 -> 8
- net /PULSE_BLATT_RAW: track 0.00 -> 86.0 mm, vias 0 -> 2
- net /PULSE_NULL_RAW: track 0.00 -> 76.9 mm
- net /AC2: track 0.00 -> 76.5 mm
- net /TRIAC_CTRL: track 0.00 -> 74.6 mm, vias 0 -> 3
- net /RS485_A: track 0.00 -> 73.5 mm, vias 0 -> 1
- net /RS485_B: track 0.00 -> 72.9 mm, vias 0 -> 1
- net /PULSE_LEER_RAW: track 0.00 -> 71.0 mm, vias 0 -> 2
- net /+15V: track 0.00 -> 67.1 mm, vias 0 -> 1
- net /+5V_IN: track 0.00 -> 66.6 mm, vias 0 -> 1
- net /AC1: track 0.00 -> 53.5 mm
- net /CHAIN_OUT_EXT: track 0.00 -> 50.2 mm, vias 0 -> 2
- net /VDRV: track 0.00 -> 39.4 mm, vias 0 -> 3
- net /TRIAC_DRV: track 0.00 -> 38.6 mm
- net /VSENS: track 0.00 -> 37.3 mm, vias 0 -> 1
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- added copper zone on B.Cu, net /GND
- added copper zone on F.Cu, net /GND
Other:
- board text added: "TenOfNine"
