File: hardware/daughtercard/daughtercard.kicad_sch (KiCad schematic)
At the start: 48 parts, among them J1 Anzeige, J2 Bus in, J3 Bus out, J4 42V~ in, J5 42V~ out, J6 UPDI, Q1 BSS84, Q2 MMBT3904, Q3 MMBT3904, U1 ATtiny1616-SNR, U2 TP8485E-SR

Commit message: JLCPCB-Bestueckung vorbereitet: LCSC-Nummern, --jlc-Export, R16 0805
- LCSC-Dict in gen_daughtercard_sch.py: Basic Parts, wo moeglich (alle
  0805/1206-R und -C, MMBT3904). Nur U1, U2 und BAT54S bleiben Extended.
- gen_daughtercard_pcb.py --jlc: erzeugt jlc/BOM.csv + jlc/CPL.csv im
  JLCPCB-Format (gitignored, Bauartefakt). Schliesst #, H*, TP*, JP*,
  J1-J6 (Handloetung) und DNP (Q3, R10) aus.
- R16 von 1206 auf 0805 (D-1): 120 Ohm gibt es bei JLCPCB nur in 0805
  als Basic Part; Verlustleistung ~50 mW unkritisch. Schaltplan und PCB
  neu erzeugt, ERC 0/0, DRC unveraendert (4 enge Nachbarpaare am
  Bus-Stecker, vom Nutzer zu justieren).
- docs/jlc-bestueckung.md: Stueckliste mit LCSC-Zuordnung, zweite
  Anschlussbild-Pruefung aller Symbole (ohne Befund: MMBT3904, BSS84,
  BAT54S, TP8485E, ATtiny1616), Ruestkosten-Bilanz, offene
  Entscheidungen D-2 (C3), D-3 (F1), D-4 (Q1-LCSC).
- schaltplan-daughtercard.md v0.4, projektstand.md, toolchain.md.

Co-Authored-By: Claude Sonnet 5 <noreply@anthropic.com>
Claude-Session: https://claude.ai/code/session_01UsXTvE3jGgoK5Hec7hVbyD
Parts:
- R16: footprint Resistor_SMD:R_1206_3216Metric -> Resistor_SMD:R_0805_2012Metric
Changed lines of the file:
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@@
 		(instances
 			(project "daughtercard"
-				(path "/d4198d74-97df-4630-b0bf-d243d277f2c6"
+				(path "/6ef3ea5c-c688-4e5d-bddc-508f0059b947"
 					(reference "U1")
 					(unit 1)
@@
 		(instances
 			(project "daughtercard"
-				(path "/d4198d74-97df-4630-b0bf-d243d277f2c6"
+				(path "/6ef3ea5c-c688-4e5d-bddc-508f0059b947"
 					(reference "U2")
 					(unit 1)
@@
 			)
 		)
-		(property "Footprint" "Resistor_SMD:R_1206_3216Metric"
+		(property "Footprint" "Resistor_SMD:R_0805_2012Metric"
 			(at 132.842 39.37 90)
 			(effects
@@
 		(instances
 			(project "daughtercard"
-				(path "/d4198d74-97df-4630-b0bf-d243d277f2c6"
+				(path "/6ef3ea5c-c688-4e5d-bddc-508f0059b947"
 					(reference "R16")
 					(unit 1)
@@
 		(instances
 			(project "daughtercard"
-				(path "/d4198d74-97df-4630-b0bf-d243d277f2c6"
+				(path "/6ef3ea5c-c688-4e5d-bddc-508f0059b947"
 					(reference "JP3")
 					(unit 1)
@@
 		(instances
 			(project "daughtercard"
-				(path "/d4198d74-97df-4630-b0bf-d243d277f2c6"
+				(path "/6ef3ea5c-c688-4e5d-bddc-508f0059b947"
 					(reference "F1")
 					(unit 1)
@@
 		(instances
 			(project "daughtercard"
-				(path "/d4198d74-97df-4630-b0bf-d243d277f2c6"
+				(path "/6ef3ea5c-c688-4e5d-bddc-508f0059b947"
 					(reference "C1")
 					(unit 1)
@@
 		(instances
 			(project "daughtercard"
-				(path "/d4198d74-97df-4630-b0bf-d243d277f2c6"
+				(path "/6ef3ea5c-c688-4e5d-bddc-508f0059b947"
 					(reference "C2")
 					(unit 1)
@@
 		(instances
 			(project "daughtercard"
-				(path "/d4198d74-97df-4630-b0bf-d243d277f2c6"
+				(path "/6ef3ea5c-c688-4e5d-bddc-508f0059b947"
 					(reference "C3")
 					(unit 1)
@@
 		(instances
 			(project "daughtercard"
-				(path "/d4198d74-97df-4630-b0bf-d243d277f2c6"
+				(path "/6ef3ea5c-c688-4e5d-bddc-508f0059b947"
 					(reference "R14")
 					(unit 1)
@@
 		(instances
 			(project "daughtercard"
-				(path "/d4198d74-97df-4630-b0bf-d243d277f2c6"
+				(path "/6ef3ea5c-c688-4e5d-bddc-508f0059b947"
 					(reference "JP1")
 					(unit 1)
@@
 		(instances
 			(project "daughtercard"
-				(path "/d4198d74-97df-4630-b0bf-d243d277f2c6"
+				(path "/6ef3ea5c-c688-4e5d-bddc-508f0059b947"
 					(reference "JP2")
 					(unit 1)
@@
 		(instances
 			(project "daughtercard"
-				(path "/d4198d74-97df-4630-b0bf-d243d277f2c6"
+				(path "/6ef3ea5c-c688-4e5d-bddc-508f0059b947"
 					(reference "Q1")
 					(unit 1)
@@
 		(instances
 			(project "daughtercard"
-				(path "/d4198d74-97df-4630-b0bf-d243d277f2c6"
+				(path "/6ef3ea5c-c688-4e5d-bddc-508f0059b947"
 					(reference "Q2")
 					(unit 1)
@@
 		(instances
 			(project "daughtercard"
-				(path "/d4198d74-97df-4630-b0bf-d243d277f2c6"
+				(path "/6ef3ea5c-c688-4e5d-bddc-508f0059b947"
 					(reference "Q3")
 					(unit 1)
@@
 		(instances
 			(project "daughtercard"
-				(path "/d4198d74-97df-4630-b0bf-d243d277f2c6"
+				(path "/6ef3ea5c-c688-4e5d-bddc-508f0059b947"
 					(reference "R7")
 					(unit 1)
@@
 		(instances
 			(project "daughtercard"
-				(path "/d4198d74-97df-4630-b0bf-d243d277f2c6"
+				(path "/6ef3ea5c-c688-4e5d-bddc-508f0059b947"
 					(reference "R8")
 					(unit 1)
@@
 		(instances
 			(project "daughtercard"
-				(path "/d4198d74-97df-4630-b0bf-d243d277f2c6"
+				(path "/6ef3ea5c-c688-4e5d-bddc-508f0059b947"
 					(reference "R9")
 					(unit 1)
@@
 		(instances
 			(project "daughtercard"
-				(path "/d4198d74-97df-4630-b0bf-d243d277f2c6"
+				(path "/6ef3ea5c-c688-4e5d-bddc-508f0059b947"
 					(reference "R10")
 					(unit 1)
@@
 		(instances
 			(project "daughtercard"
-				(path "/d4198d74-97df-4630-b0bf-d243d277f2c6"
+				(path "/6ef3ea5c-c688-4e5d-bddc-508f0059b947"
 					(reference "R1")
 					(unit 1)
@@
 		(instances
 			(project "daughtercard"
-				(path "/d4198d74-97df-4630-b0bf-d243d277f2c6"
+				(path "/6ef3ea5c-c688-4e5d-bddc-508f0059b947"
 					(reference "R2")
 					(unit 1)
@@
 		(instances
 			(project "daughtercard"
-				(path "/d4198d74-97df-4630-b0bf-d243d277f2c6"
+				(path "/6ef3ea5c-c688-4e5d-bddc-508f0059b947"
 					(reference "C4")
 					(unit 1)
@@
 		(instances
 			(project "daughtercard"
-				(path "/d4198d74-97df-4630-b0bf-d243d277f2c6"
+				(path "/6ef3ea5c-c688-4e5d-bddc-508f0059b947"
 					(reference "D1")
 					(unit 1)
@@
 		(instances
 			(project "daughtercard"
-				(path "/d4198d74-97df-4630-b0bf-d243d277f2c6"
+				(path "/6ef3ea5c-c688-4e5d-bddc-508f0059b947"
 					(reference "R3")
 					(unit 1)
@@
 		(instances
 			(project "daughtercard"
-				(path "/d4198d74-97df-4630-b0bf-d243d277f2c6"
+				(path "/6ef3ea5c-c688-4e5d-bddc-508f0059b947"
 					(reference "R4")
 					(unit 1)
@@
 		(instances
 			(project "daughtercard"
-				(path "/d4198d74-97df-4630-b0bf-d243d277f2c6"
+				(path "/6ef3ea5c-c688-4e5d-bddc-508f0059b947"
 					(reference "C5")
 					(unit 1)
@@
 		(instances
 			(project "daughtercard"
-				(path "/d4198d74-97df-4630-b0bf-d243d277f2c6"
+				(path "/6ef3ea5c-c688-4e5d-bddc-508f0059b947"
 					(reference "D2")
 					(unit 1)
@@
 		(instances
 			(project "daughtercard"
-				(path "/d4198d74-97df-4630-b0bf-d243d277f2c6"
+				(path "/6ef3ea5c-c688-4e5d-bddc-508f0059b947"
 					(reference "R5")
 					(unit 1)
@@
 		(instances
 			(project "daughtercard"
-				(path "/d4198d74-97df-4630-b0bf-d243d277f2c6"
+				(path "/6ef3ea5c-c688-4e5d-bddc-508f0059b947"
 					(reference "R6")
 					(unit 1)
@@
 		(instances
 			(project "daughtercard"
-				(path "/d4198d74-97df-4630-b0bf-d243d277f2c6"
+				(path "/6ef3ea5c-c688-4e5d-bddc-508f0059b947"
 					(reference "C6")
 					(unit 1)
@@
 		(instances
 			(project "daughtercard"
-				(path "/d4198d74-97df-4630-b0bf-d243d277f2c6"
+				(path "/6ef3ea5c-c688-4e5d-bddc-508f0059b947"
 					(reference "D3")
 					(unit 1)
@@
 		(instances
 			(project "daughtercard"
-				(path "/d4198d74-97df-4630-b0bf-d243d277f2c6"
+				(path "/6ef3ea5c-c688-4e5d-bddc-508f0059b947"
 					(reference "R11")
 					(unit 1)
@@
 		(instances
 			(project "daughtercard"
-				(path "/d4198d74-97df-4630-b0bf-d243d277f2c6"
+				(path "/6ef3ea5c-c688-4e5d-bddc-508f0059b947"
 					(reference "R12")
 					(unit 1)
@@
 		(instances
 			(project "daughtercard"
-				(path "/d4198d74-97df-4630-b0bf-d243d277f2c6"
+				(path "/6ef3ea5c-c688-4e5d-bddc-508f0059b947"
 					(reference "R13")
 					(unit 1)
@@
 		(instances
 			(project "daughtercard"
-				(path "/d4198d74-97df-4630-b0bf-d243d277f2c6"
+				(path "/6ef3ea5c-c688-4e5d-bddc-508f0059b947"
 					(reference "R15")
 					(unit 1)
@@
 		(instances
 			(project "daughtercard"
-				(path "/d4198d74-97df-4630-b0bf-d243d277f2c6"
+				(path "/6ef3ea5c-c688-4e5d-bddc-508f0059b947"
 					(reference "D4")
 					(unit 1)
@@
 		(instances
 			(project "daughtercard"
-				(path "/d4198d74-97df-4630-b0bf-d243d277f2c6"
+				(path "/6ef3ea5c-c688-4e5d-bddc-508f0059b947"
 					(reference "J6")
 					(unit 1)
@@
 		(instances
 			(project "daughtercard"
-				(path "/d4198d74-97df-4630-b0bf-d243d277f2c6"
+				(path "/6ef3ea5c-c688-4e5d-bddc-508f0059b947"
 					(reference "J1")
 					(unit 1)
@@
 		(instances
 			(project "daughtercard"
-				(path "/d4198d74-97df-4630-b0bf-d243d277f2c6"
+				(path "/6ef3ea5c-c688-4e5d-bddc-508f0059b947"
 					(reference "J2")
 					(unit 1)
@@
 		(instances
 			(project "daughtercard"
-				(path "/d4198d74-97df-4630-b0bf-d243d277f2c6"
+				(path "/6ef3ea5c-c688-4e5d-bddc-508f0059b947"
 					(reference "J3")
 					(unit 1)
@@
 		(instances
 			(project "daughtercard"
-				(path "/d4198d74-97df-4630-b0bf-d243d277f2c6"
+				(path "/6ef3ea5c-c688-4e5d-bddc-508f0059b947"
 					(reference "J4")
 					(unit 1)
@@
 		(instances
 			(project "daughtercard"
-				(path "/d4198d74-97df-4630-b0bf-d243d277f2c6"
+				(path "/6ef3ea5c-c688-4e5d-bddc-508f0059b947"
 					(reference "J5")
 					(unit 1)
@@
 		(instances
 			(project "daughtercard"
-				(path "/d4198d74-97df-4630-b0bf-d243d277f2c6"
+				(path "/6ef3ea5c-c688-4e5d-bddc-508f0059b947"
 					(reference "TP1")
 					(unit 1)
@@
 		(instances
 			(project "daughtercard"
-				(path "/d4198d74-97df-4630-b0bf-d243d277f2c6"
+				(path "/6ef3ea5c-c688-4e5d-bddc-508f0059b947"
 					(reference "TP2")
 					(unit 1)
@@
 		(instances
 			(project "daughtercard"
-				(path "/d4198d74-97df-4630-b0bf-d243d277f2c6"
+				(path "/6ef3ea5c-c688-4e5d-bddc-508f0059b947"
 					(reference "TP3")
 					(unit 1)
@@
 		(instances
 			(project "daughtercard"
-				(path "/d4198d74-97df-4630-b0bf-d243d277f2c6"
+				(path "/6ef3ea5c-c688-4e5d-bddc-508f0059b947"
 					(reference "TP4")
 					(unit 1)
@@
 		(instances
 			(project "daughtercard"
-				(path "/d4198d74-97df-4630-b0bf-d243d277f2c6"
+				(path "/6ef3ea5c-c688-4e5d-bddc-508f0059b947"
 					(reference "TP5")
 					(unit 1)
@@
 		(instances
 			(project "daughtercard"
-				(path "/d4198d74-97df-4630-b0bf-d243d277f2c6"
+				(path "/6ef3ea5c-c688-4e5d-bddc-508f0059b947"
 					(reference "TP6")
 					(unit 1)
@@
 		(instances
 			(project "daughtercard"
-				(path "/d4198d74-97df-4630-b0bf-d243d277f2c6"
+				(path "/6ef3ea5c-c688-4e5d-bddc-508f0059b947"
 					(reference "TP7")
 					(unit 1)
@@
 		(instances
 			(project "daughtercard"
-				(path "/d4198d74-97df-4630-b0bf-d243d277f2c6"
+				(path "/6ef3ea5c-c688-4e5d-bddc-508f0059b947"
 					(reference "#FLG1")
 					(unit 1)
@@
 		(instances
 			(project "daughtercard"
-				(path "/d4198d74-97df-4630-b0bf-d243d277f2c6"
+				(path "/6ef3ea5c-c688-4e5d-bddc-508f0059b947"
 					(reference "#FLG2")
 					(unit 1)
@@
 		(instances
 			(project "daughtercard"
-				(path "/d4198d74-97df-4630-b0bf-d243d277f2c6"
+				(path "/6ef3ea5c-c688-4e5d-bddc-508f0059b947"
 					(reference "#FLG3")
 					(unit 1)
@@
 		(instances
 			(project "daughtercard"
-				(path "/d4198d74-97df-4630-b0bf-d243d277f2c6"
+				(path "/6ef3ea5c-c688-4e5d-bddc-508f0059b947"
 					(reference "#FLG4")
 					(unit 1)

Commit message: J1 von Wannenstecker auf Buchsenleiste 2x5 (board-to-board)
Die Daughter Card wird huckepack direkt auf den Pfostenstecker der
Anzeigenplatine gesteckt (Ruecksprache 31.08.2026). Ein Wannenstecker
(Stifte im Kragen) passt dort nicht - richtig ist eine Buchsenleiste.

- Footprint J1: Connector_IDC:IDC-Header_2x05_P2.54mm_Vertical
  -> Connector_PinSocket_2.54mm:PinSocket_2x05_P2.54mm_Vertical
  (Referenz BKL 10120960). Pinbelegung 1..10 unveraendert.
- J1 ist damit NICHT mehr mechanisch kodiert. Pin 2/4 fuehren 42 V~;
  180-Grad-verdreht aufgesteckt zerstoert das U1/U2/Q1/Q2. Abgesichert
  ueber Mechanik (offen: J1-M), Bestueckungsdruck und Durchgangspruefung.
- docs/pruefpunkte-j1-buchsenleiste.md: Bewertung, Absicherung, Freigabe,
  offener Punkt J1-M (mechanische Kodierung der Drehlage).
- Schaltplan v0.5 (4.1 Verpol-Hinweis, 3.3, Pruefliste 9.1),
  Spezifikation v0.8 (4.6), layout-daughtercard.md (Checkliste, AC-Zone,
  Courtyard-Notiz), projektstand.md.
- Schaltplan + PCB neu erzeugt, ERC 0/0, DRC unveraendert (4 enge Paare
  am Bus-Stecker J2/J3, nichts an J1).

Co-Authored-By: Claude Sonnet 5 <noreply@anthropic.com>
Claude-Session: https://claude.ai/code/session_01UsXTvE3jGgoK5Hec7hVbyD
Parts:
- J1: footprint Connector_IDC:IDC-Header_2x05_P2.54mm_Vertical -> Connector_PinSocket_2.54mm:PinSocket_2x05_P2.54mm_Vertical
Changed lines of the file:
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@@
 		(instances
 			(project "daughtercard"
-				(path "/6ef3ea5c-c688-4e5d-bddc-508f0059b947"
+				(path "/e1c88223-9aeb-41d2-aa44-249e62b8a058"
 					(reference "U1")
 					(unit 1)
@@
 		(instances
 			(project "daughtercard"
-				(path "/6ef3ea5c-c688-4e5d-bddc-508f0059b947"
+				(path "/e1c88223-9aeb-41d2-aa44-249e62b8a058"
 					(reference "U2")
 					(unit 1)
@@
 		(instances
 			(project "daughtercard"
-				(path "/6ef3ea5c-c688-4e5d-bddc-508f0059b947"
+				(path "/e1c88223-9aeb-41d2-aa44-249e62b8a058"
 					(reference "R16")
 					(unit 1)
@@
 		(instances
 			(project "daughtercard"
-				(path "/6ef3ea5c-c688-4e5d-bddc-508f0059b947"
+				(path "/e1c88223-9aeb-41d2-aa44-249e62b8a058"
 					(reference "JP3")
 					(unit 1)
@@
 		(instances
 			(project "daughtercard"
-				(path "/6ef3ea5c-c688-4e5d-bddc-508f0059b947"
+				(path "/e1c88223-9aeb-41d2-aa44-249e62b8a058"
 					(reference "F1")
 					(unit 1)
@@
 		(instances
 			(project "daughtercard"
-				(path "/6ef3ea5c-c688-4e5d-bddc-508f0059b947"
+				(path "/e1c88223-9aeb-41d2-aa44-249e62b8a058"
 					(reference "C1")
 					(unit 1)
@@
 		(instances
 			(project "daughtercard"
-				(path "/6ef3ea5c-c688-4e5d-bddc-508f0059b947"
+				(path "/e1c88223-9aeb-41d2-aa44-249e62b8a058"
 					(reference "C2")
 					(unit 1)
@@
 		(instances
 			(project "daughtercard"
-				(path "/6ef3ea5c-c688-4e5d-bddc-508f0059b947"
+				(path "/e1c88223-9aeb-41d2-aa44-249e62b8a058"
 					(reference "C3")
 					(unit 1)
@@
 		(instances
 			(project "daughtercard"
-				(path "/6ef3ea5c-c688-4e5d-bddc-508f0059b947"
+				(path "/e1c88223-9aeb-41d2-aa44-249e62b8a058"
 					(reference "R14")
 					(unit 1)
@@
 		(instances
 			(project "daughtercard"
-				(path "/6ef3ea5c-c688-4e5d-bddc-508f0059b947"
+				(path "/e1c88223-9aeb-41d2-aa44-249e62b8a058"
 					(reference "JP1")
 					(unit 1)
@@
 		(instances
 			(project "daughtercard"
-				(path "/6ef3ea5c-c688-4e5d-bddc-508f0059b947"
+				(path "/e1c88223-9aeb-41d2-aa44-249e62b8a058"
 					(reference "JP2")
 					(unit 1)
@@
 		(instances
 			(project "daughtercard"
-				(path "/6ef3ea5c-c688-4e5d-bddc-508f0059b947"
+				(path "/e1c88223-9aeb-41d2-aa44-249e62b8a058"
 					(reference "Q1")
 					(unit 1)
@@
 		(instances
 			(project "daughtercard"
-				(path "/6ef3ea5c-c688-4e5d-bddc-508f0059b947"
+				(path "/e1c88223-9aeb-41d2-aa44-249e62b8a058"
 					(reference "Q2")
 					(unit 1)
@@
 		(instances
 			(project "daughtercard"
-				(path "/6ef3ea5c-c688-4e5d-bddc-508f0059b947"
+				(path "/e1c88223-9aeb-41d2-aa44-249e62b8a058"
 					(reference "Q3")
 					(unit 1)
@@
 		(instances
 			(project "daughtercard"
-				(path "/6ef3ea5c-c688-4e5d-bddc-508f0059b947"
+				(path "/e1c88223-9aeb-41d2-aa44-249e62b8a058"
 					(reference "R7")
 					(unit 1)
@@
 		(instances
 			(project "daughtercard"
-				(path "/6ef3ea5c-c688-4e5d-bddc-508f0059b947"
+				(path "/e1c88223-9aeb-41d2-aa44-249e62b8a058"
 					(reference "R8")
 					(unit 1)
@@
 		(instances
 			(project "daughtercard"
-				(path "/6ef3ea5c-c688-4e5d-bddc-508f0059b947"
+				(path "/e1c88223-9aeb-41d2-aa44-249e62b8a058"
 					(reference "R9")
 					(unit 1)
@@
 		(instances
 			(project "daughtercard"
-				(path "/6ef3ea5c-c688-4e5d-bddc-508f0059b947"
+				(path "/e1c88223-9aeb-41d2-aa44-249e62b8a058"
 					(reference "R10")
 					(unit 1)
@@
 		(instances
 			(project "daughtercard"
-				(path "/6ef3ea5c-c688-4e5d-bddc-508f0059b947"
+				(path "/e1c88223-9aeb-41d2-aa44-249e62b8a058"
 					(reference "R1")
 					(unit 1)
@@
 		(instances
 			(project "daughtercard"
-				(path "/6ef3ea5c-c688-4e5d-bddc-508f0059b947"
+				(path "/e1c88223-9aeb-41d2-aa44-249e62b8a058"
 					(reference "R2")
 					(unit 1)
@@
 		(instances
 			(project "daughtercard"
-				(path "/6ef3ea5c-c688-4e5d-bddc-508f0059b947"
+				(path "/e1c88223-9aeb-41d2-aa44-249e62b8a058"
 					(reference "C4")
 					(unit 1)
@@
 		(instances
 			(project "daughtercard"
-				(path "/6ef3ea5c-c688-4e5d-bddc-508f0059b947"
+				(path "/e1c88223-9aeb-41d2-aa44-249e62b8a058"
 					(reference "D1")
 					(unit 1)
@@
 		(instances
 			(project "daughtercard"
-				(path "/6ef3ea5c-c688-4e5d-bddc-508f0059b947"
+				(path "/e1c88223-9aeb-41d2-aa44-249e62b8a058"
 					(reference "R3")
 					(unit 1)
@@
 		(instances
 			(project "daughtercard"
-				(path "/6ef3ea5c-c688-4e5d-bddc-508f0059b947"
+				(path "/e1c88223-9aeb-41d2-aa44-249e62b8a058"
 					(reference "R4")
 					(unit 1)
@@
 		(instances
 			(project "daughtercard"
-				(path "/6ef3ea5c-c688-4e5d-bddc-508f0059b947"
+				(path "/e1c88223-9aeb-41d2-aa44-249e62b8a058"
 					(reference "C5")
 					(unit 1)
@@
 		(instances
 			(project "daughtercard"
-				(path "/6ef3ea5c-c688-4e5d-bddc-508f0059b947"
+				(path "/e1c88223-9aeb-41d2-aa44-249e62b8a058"
 					(reference "D2")
 					(unit 1)
@@
 		(instances
 			(project "daughtercard"
-				(path "/6ef3ea5c-c688-4e5d-bddc-508f0059b947"
+				(path "/e1c88223-9aeb-41d2-aa44-249e62b8a058"
 					(reference "R5")
 					(unit 1)
@@
 		(instances
 			(project "daughtercard"
-				(path "/6ef3ea5c-c688-4e5d-bddc-508f0059b947"
+				(path "/e1c88223-9aeb-41d2-aa44-249e62b8a058"
 					(reference "R6")
 					(unit 1)
@@
 		(instances
 			(project "daughtercard"
-				(path "/6ef3ea5c-c688-4e5d-bddc-508f0059b947"
+				(path "/e1c88223-9aeb-41d2-aa44-249e62b8a058"
 					(reference "C6")
 					(unit 1)
@@
 		(instances
 			(project "daughtercard"
-				(path "/6ef3ea5c-c688-4e5d-bddc-508f0059b947"
+				(path "/e1c88223-9aeb-41d2-aa44-249e62b8a058"
 					(reference "D3")
 					(unit 1)
@@
 		(instances
 			(project "daughtercard"
-				(path "/6ef3ea5c-c688-4e5d-bddc-508f0059b947"
+				(path "/e1c88223-9aeb-41d2-aa44-249e62b8a058"
 					(reference "R11")
 					(unit 1)
@@
 		(instances
 			(project "daughtercard"
-				(path "/6ef3ea5c-c688-4e5d-bddc-508f0059b947"
+				(path "/e1c88223-9aeb-41d2-aa44-249e62b8a058"
 					(reference "R12")
 					(unit 1)
@@
 		(instances
 			(project "daughtercard"
-				(path "/6ef3ea5c-c688-4e5d-bddc-508f0059b947"
+				(path "/e1c88223-9aeb-41d2-aa44-249e62b8a058"
 					(reference "R13")
 					(unit 1)
@@
 		(instances
 			(project "daughtercard"
-				(path "/6ef3ea5c-c688-4e5d-bddc-508f0059b947"
+				(path "/e1c88223-9aeb-41d2-aa44-249e62b8a058"
 					(reference "R15")
 					(unit 1)
@@
 		(instances
 			(project "daughtercard"
-				(path "/6ef3ea5c-c688-4e5d-bddc-508f0059b947"
+				(path "/e1c88223-9aeb-41d2-aa44-249e62b8a058"
 					(reference "D4")
 					(unit 1)
@@
 		(instances
 			(project "daughtercard"
-				(path "/6ef3ea5c-c688-4e5d-bddc-508f0059b947"
+				(path "/e1c88223-9aeb-41d2-aa44-249e62b8a058"
 					(reference "J6")
 					(unit 1)
@@
 			)
 		)
-		(property "Footprint" "Connector_IDC:IDC-Header_2x05_P2.54mm_Vertical"
+		(property "Footprint" "Connector_PinSocket_2.54mm:PinSocket_2x05_P2.54mm_Vertical"
 			(at 25.4 299.72 0.0000)
 			(effects
@@
 		(instances
 			(project "daughtercard"
-				(path "/6ef3ea5c-c688-4e5d-bddc-508f0059b947"
+				(path "/e1c88223-9aeb-41d2-aa44-249e62b8a058"
 					(reference "J1")
 					(unit 1)
@@
 		(instances
 			(project "daughtercard"
-				(path "/6ef3ea5c-c688-4e5d-bddc-508f0059b947"
+				(path "/e1c88223-9aeb-41d2-aa44-249e62b8a058"
 					(reference "J2")
 					(unit 1)
@@
 		(instances
 			(project "daughtercard"
-				(path "/6ef3ea5c-c688-4e5d-bddc-508f0059b947"
+				(path "/e1c88223-9aeb-41d2-aa44-249e62b8a058"
 					(reference "J3")
 					(unit 1)
@@
 		(instances
 			(project "daughtercard"
-				(path "/6ef3ea5c-c688-4e5d-bddc-508f0059b947"
+				(path "/e1c88223-9aeb-41d2-aa44-249e62b8a058"
 					(reference "J4")
 					(unit 1)
@@
 		(instances
 			(project "daughtercard"
-				(path "/6ef3ea5c-c688-4e5d-bddc-508f0059b947"
+				(path "/e1c88223-9aeb-41d2-aa44-249e62b8a058"
 					(reference "J5")
 					(unit 1)
@@
 		(instances
 			(project "daughtercard"
-				(path "/6ef3ea5c-c688-4e5d-bddc-508f0059b947"
+				(path "/e1c88223-9aeb-41d2-aa44-249e62b8a058"
 					(reference "TP1")
 					(unit 1)
@@
 		(instances
 			(project "daughtercard"
-				(path "/6ef3ea5c-c688-4e5d-bddc-508f0059b947"
+				(path "/e1c88223-9aeb-41d2-aa44-249e62b8a058"
 					(reference "TP2")
 					(unit 1)
@@
 		(instances
 			(project "daughtercard"
-				(path "/6ef3ea5c-c688-4e5d-bddc-508f0059b947"
+				(path "/e1c88223-9aeb-41d2-aa44-249e62b8a058"
 					(reference "TP3")
 					(unit 1)
@@
 		(instances
 			(project "daughtercard"
-				(path "/6ef3ea5c-c688-4e5d-bddc-508f0059b947"
+				(path "/e1c88223-9aeb-41d2-aa44-249e62b8a058"
 					(reference "TP4")
 					(unit 1)
@@
 		(instances
 			(project "daughtercard"
-				(path "/6ef3ea5c-c688-4e5d-bddc-508f0059b947"
+				(path "/e1c88223-9aeb-41d2-aa44-249e62b8a058"
 					(reference "TP5")
 					(unit 1)
@@
 		(instances
 			(project "daughtercard"
-				(path "/6ef3ea5c-c688-4e5d-bddc-508f0059b947"
+				(path "/e1c88223-9aeb-41d2-aa44-249e62b8a058"
 					(reference "TP6")
 					(unit 1)
@@
 		(instances
 			(project "daughtercard"
-				(path "/6ef3ea5c-c688-4e5d-bddc-508f0059b947"
+				(path "/e1c88223-9aeb-41d2-aa44-249e62b8a058"
 					(reference "TP7")
 					(unit 1)
@@
 		(instances
 			(project "daughtercard"
-				(path "/6ef3ea5c-c688-4e5d-bddc-508f0059b947"
+				(path "/e1c88223-9aeb-41d2-aa44-249e62b8a058"
 					(reference "#FLG1")
 					(unit 1)
@@
 		(instances
 			(project "daughtercard"
-				(path "/6ef3ea5c-c688-4e5d-bddc-508f0059b947"
+				(path "/e1c88223-9aeb-41d2-aa44-249e62b8a058"
 					(reference "#FLG2")
 					(unit 1)
@@
 		(instances
 			(project "daughtercard"
-				(path "/6ef3ea5c-c688-4e5d-bddc-508f0059b947"
+				(path "/e1c88223-9aeb-41d2-aa44-249e62b8a058"
 					(reference "#FLG3")
 					(unit 1)
@@
 		(instances
 			(project "daughtercard"
-				(path "/6ef3ea5c-c688-4e5d-bddc-508f0059b947"
+				(path "/e1c88223-9aeb-41d2-aa44-249e62b8a058"
 					(reference "#FLG4")
 					(unit 1)
